File: hardware/bldc-controller.kicad_pcb (KiCad board)
At the start: 4 copper layers, 60 x 60 mm, 369 parts, among them J1 USB_MICRO_B, J2 JST GH, J3 JST GH, J4 1.27mm Pin Header, J5 JST GH, J6 JST GH, P1 Solder Terminal, P2 Solder Terminal, P3 Solder Terminal, P4 Solder Terminal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

Commit message: Rev. B hardware design files
Parts:
- P1, P2, P3, P4, P5: footprint bldc-controller:SOLDER_PAD -> bldc-controller:SOLDER_HOLE_1.5MM
- Q1, Q2, Q3, Q4, Q5, Q6: value CSD18540Q5B -> CSD18533
- R10, R11, R16, R17, R22, R23: value TBD -> 4.7
- U3, U4, U5: value INA240A1 -> INA240A2
Routing:
- net /Half Bridge B/PHASE: track 41.8 -> 43.9 mm
- net /Half Bridge A/PHASE: track 33.2 -> 35.3 mm
- net /Half Bridge C/PHASE: track 49.4 -> 51.6 mm
Other:
- rule pad_to_mask_clearance: 0.0762 -> 0.0508
- board text added: "9/2017"
- board text added: "BLDC Servo Controller rev. B"
- board text added: "BLDC rev. B"
- board text removed: "8/2017"
- board text removed: "BLDC Servo Controller rev. A"
- board text removed: "BLDC rev. A"
